File: F7&UI&keyholder.sch (EAGLE design)
At the start: 46 parts, among them IC2 LTC485N, IC4 MCP2561-E_P

Commit message: #update UI,F7 シルク官僚
Parts:
- IC2: device linear-technology:LTC485N -> 0linear-technology:LTC485N
- renumbered TO-F7 to TO-MAIN, TO-UI3 to TO-MAIN2
Changed lines of the file:
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@@
 <part name="U$1" library="F7-DISCO" deviceset="F7-DISCO-ARDUINO" device=""/>
 <part name="IC4" library="MCP2561-E_P" deviceset="MCP2561-E_P" device=""/>
-<part name="IC2" library="linear-technology" library_urn="urn:adsk.eagle:library:261" deviceset="LTC485" device="N" package3d_urn="urn:adsk.eagle:package:16059/1"/>
-<part name="TO-F7" library="0con-harting-ml" deviceset="ML14" device=""/>
+<part name="IC2" library="0linear-technology" deviceset="LTC485" device="N" package3d_urn="urn:adsk.eagle:package:16059/1"/>
+<part name="TO-MAIN" library="0con-harting-ml" deviceset="ML14" device=""/>
 <part name="GND44" library="supply1" deviceset="GND" device=""/>
 <part name="GND1" library="supply1" deviceset="GND" device=""/>
@@
 <part name="SUPPLY10" library="supply2" library_urn="urn:adsk.eagle:library:372" deviceset="GND2" device=""/>
 <part name="VDD3" library="supply1" library_urn="urn:adsk.eagle:library:371" deviceset="VDD" device=""/>
-<part name="TO-UI3" library="0con-harting-ml" deviceset="ML14" device=""/>
+<part name="TO-MAIN2" library="0con-harting-ml" deviceset="ML14" device=""/>
 <part name="VDD4" library="supply1" library_urn="urn:adsk.eagle:library:371" deviceset="VDD" device=""/>
 <part name="SUPPLY12" library="supply2" library_urn="urn:adsk.eagle:library:372" deviceset="GND2" device=""/>
@@
 <attribute name="VALUE" x="-5.08" y="45.72" size="1.778" layer="96"/>
 </instance>
-<instance part="TO-F7" gate="1" x="154.94" y="12.7" smashed="yes">
+<instance part="TO-MAIN" gate="1" x="154.94" y="12.7" smashed="yes">
 <attribute name="VALUE" x="151.13" y="0" size="1.778" layer="96"/>
 <attribute name="NAME" x="151.13" y="23.622" size="1.778" layer="95"/>
@@
 </instance>
 <instance part="VDD3" gate="G$1" x="427.355" y="98.1075" smashed="yes" rot="R270"/>
-<instance part="TO-UI3" gate="1" x="418.465" y="17.4625" smashed="yes">
+<instance part="TO-MAIN2" gate="1" x="418.465" y="17.4625" smashed="yes">
 <attribute name="VALUE" x="414.655" y="7.3025" size="1.778" layer="96"/>
 <attribute name="NAME" x="414.655" y="25.8445" size="1.778" layer="95"/>
@@
 <net name="+12V" class="0">
 <segment>
-<pinref part="TO-F7" gate="1" pin="14"/>
+<pinref part="TO-MAIN" gate="1" pin="14"/>
 <wire x1="147.32" y1="20.32" x2="142.24" y2="20.32" width="0.1524" layer="91"/>
 <wire x1="142.24" y1="20.32" x2="142.24" y2="27.94" width="0.1524" layer="91"/>
@@
 <net name="GND" class="0">
 <segment>
-<pinref part="TO-F7" gate="1" pin="1"/>
+<pinref part="TO-MAIN" gate="1" pin="1"/>
 <wire x1="162.56" y1="5.08" x2="167.64" y2="5.08" width="0.1524" layer="91"/>
 <wire x1="167.64" y1="5.08" x2="167.64" y2="-5.08" width="0.1524" layer="91"/>
@@
 <net name="RS-CHB" class="0">
 <segment>
-<pinref part="TO-F7" gate="1" pin="5"/>
+<pinref part="TO-MAIN" gate="1" pin="5"/>
 <wire x1="162.56" y1="10.16" x2="167.64" y2="10.16" width="0.1524" layer="91"/>
 <label x="167.64" y="10.16" size="1.27" layer="95" xref="yes"/>
@@
 <net name="RS-CHA" class="0">
 <segment>
-<pinref part="TO-F7" gate="1" pin="6"/>
+<pinref part="TO-MAIN" gate="1" pin="6"/>
 <wire x1="147.32" y1="10.16" x2="139.7" y2="10.16" width="0.1524" layer="91"/>
 <label x="139.7" y="10.16" size="1.27" layer="95" rot="R180" xref="yes"/>
@@
 <net name="EMERGENCY" class="0">
 <segment>
-<pinref part="TO-F7" gate="1" pin="2"/>
+<pinref part="TO-MAIN" gate="1" pin="2"/>
 <wire x1="147.32" y1="5.08" x2="142.24" y2="5.08" width="0.1524" layer="91"/>
 <label x="142.24" y="5.08" size="1.27" layer="95" rot="R180" xref="yes"/>
@@
 <net name="F7-F4-SIG1" class="0">
 <segment>
-<pinref part="TO-F7" gate="1" pin="12"/>
+<pinref part="TO-MAIN" gate="1" pin="12"/>
 <wire x1="139.7" y1="17.78" x2="147.32" y2="17.78" width="0.1524" layer="91"/>
 <label x="139.7" y="17.78" size="1.27" layer="95" rot="R180" xref="yes"/>
@@
 <net name="F7-F4-SIG2" class="0">
 <segment>
-<pinref part="TO-F7" gate="1" pin="11"/>
+<pinref part="TO-MAIN" gate="1" pin="11"/>
 <wire x1="162.56" y1="17.78" x2="167.64" y2="17.78" width="0.1524" layer="91"/>
 <label x="167.64" y="17.78" size="1.27" layer="95" xref="yes"/>
@@
 <net name="F7-RS-SIG1" class="0">
 <segment>
-<pinref part="TO-F7" gate="1" pin="10"/>
+<pinref part="TO-MAIN" gate="1" pin="10"/>
 <wire x1="139.7" y1="15.24" x2="147.32" y2="15.24" width="0.1524" layer="91"/>
 <label x="139.7" y="15.24" size="1.27" layer="95" rot="R180" xref="yes"/>
@@
 <net name="F7-RS-SIG2" class="0">
 <segment>
-<pinref part="TO-F7" gate="1" pin="9"/>
+<pinref part="TO-MAIN" gate="1" pin="9"/>
 <wire x1="162.56" y1="15.24" x2="167.64" y2="15.24" width="0.1524" layer="91"/>
 <label x="167.64" y="15.24" size="1.27" layer="95" xref="yes"/>
@@
 <net name="LIPO" class="0">
 <segment>
-<pinref part="TO-F7" gate="1" pin="13"/>
+<pinref part="TO-MAIN" gate="1" pin="13"/>
 <wire x1="162.56" y1="20.32" x2="167.64" y2="20.32" width="0.1524" layer="91"/>
 <wire x1="167.64" y1="20.32" x2="167.64" y2="27.94" width="0.1524" layer="91"/>
@@
 <net name="HUMAN1" class="0">
 <segment>
-<pinref part="TO-F7" gate="1" pin="4"/>
+<pinref part="TO-MAIN" gate="1" pin="4"/>
 <wire x1="147.32" y1="7.62" x2="139.7" y2="7.62" width="0.1524" layer="91"/>
 <label x="139.7" y="7.62" size="1.27" layer="95" rot="R180" xref="yes"/>
@@
 <net name="CAN-L" class="0">
 <segment>
-<pinref part="TO-F7" gate="1" pin="7"/>
+<pinref part="TO-MAIN" gate="1" pin="7"/>
 <wire x1="162.56" y1="12.7" x2="167.64" y2="12.7" width="0.1524" layer="91"/>
 <label x="167.64" y="12.7" size="1.27" layer="95" xref="yes"/>
@@
 <net name="CAN-H" class="0">
 <segment>
-<pinref part="TO-F7" gate="1" pin="8"/>
+<pinref part="TO-MAIN" gate="1" pin="8"/>
 <wire x1="139.7" y1="12.7" x2="147.32" y2="12.7" width="0.1524" layer="91"/>
 <label x="139.7" y="12.7" size="1.27" layer="95" rot="R180" xref="yes"/>
@@
 <wire x1="405.4475" y1="17.4625" x2="410.845" y2="17.4625" width="0.1524" layer="91"/>
 <label x="405.4475" y="17.4625" size="1.27" layer="95" rot="R180" xref="yes"/>
-<pinref part="TO-UI3" gate="1" pin="8"/>
+<pinref part="TO-MAIN2" gate="1" pin="8"/>
 </segment>
 </net>
@@
 <wire x1="426.085" y1="22.5425" x2="433.705" y2="22.5425" width="0.1524" layer="91"/>
 <label x="433.705" y="22.5425" size="1.27" layer="95" xref="yes"/>
-<pinref part="TO-UI3" gate="1" pin="11"/>
+<pinref part="TO-MAIN2" gate="1" pin="11"/>
 </segment>
 </net>
@@
 <wire x1="410.845" y1="20.0025" x2="405.765" y2="20.0025" width="0.1524" layer="91"/>
 <label x="405.765" y="20.0025" size="1.27" layer="95" rot="R180" xref="yes"/>
-<pinref part="TO-UI3" gate="1" pin="10"/>
+<pinref part="TO-MAIN2" gate="1" pin="10"/>
 </segment>
 </net>
@@
 <wire x1="433.705" y1="20.0025" x2="426.085" y2="20.0025" width="0.1524" layer="91"/>
 <label x="433.705" y="20.0025" size="1.27" layer="95" xref="yes"/>
-<pinref part="TO-UI3" gate="1" pin="9"/>
+<pinref part="TO-MAIN2" gate="1" pin="9"/>
 </segment>
 </net>
@@
 </segment>
 <segment>
-<pinref part="TO-UI3" gate="1" pin="13"/>
+<pinref part="TO-MAIN2" gate="1" pin="13"/>
 <wire x1="429.514" y1="25.146" x2="426.085" y2="25.146" width="0.1524" layer="91"/>
 <wire x1="426.085" y1="25.146" x2="426.085" y2="25.0825" width="0.1524" layer="91"/>
@@
 </segment>
 <segment>
-<pinref part="TO-UI3" gate="1" pin="6"/>
+<pinref part="TO-MAIN2" gate="1" pin="6"/>
 <wire x1="410.845" y1="14.9225" x2="405.765" y2="14.9225" width="0.1524" layer="91"/>
 <label x="405.765" y="14.9225" size="1.27" layer="95" rot="R180" xref="yes"/>
@@
 <wire x1="431.165" y1="14.9225" x2="426.085" y2="14.9225" width="0.1524" layer="91"/>
 <label x="431.165" y="14.9225" size="1.27" layer="95" xref="yes"/>
-<pinref part="TO-UI3" gate="1" pin="5"/>
+<pinref part="TO-MAIN2" gate="1" pin="5"/>
 </segment>
 </net>
@@
 </segment>
 <segment>
-<pinref part="TO-UI3" gate="1" pin="7"/>
+<pinref part="TO-MAIN2" gate="1" pin="7"/>
 <wire x1="426.085" y1="17.4625" x2="431.165" y2="17.4625" width="0.1524" layer="91"/>
 <label x="431.165" y="17.4625" size="1.27" layer="95" xref="yes"/>
@@
 <wire x1="410.845" y1="22.5425" x2="405.765" y2="22.5425" width="0.1524" layer="91"/>
 <label x="405.765" y="22.5425" size="1.27" layer="95" rot="R180" xref="yes"/>
-<pinref part="TO-UI3" gate="1" pin="12"/>
+<pinref part="TO-MAIN2" gate="1" pin="12"/>
 </segment>
 <segment>
@@
 <net name="+12VS" class="0">
 <segment>
-<pinref part="TO-UI3" gate="1" pin="3"/>
+<pinref part="TO-MAIN2" gate="1" pin="3"/>
 <wire x1="426.085" y1="12.3825" x2="431.165" y2="12.3825" width="0.1524" layer="91"/>
 <label x="431.165" y="12.3825" size="1.27" layer="95" xref="yes"/>
@@
 <net name="MOTOR-FET" class="0">
 <segment>
-<pinref part="TO-UI3" gate="1" pin="2"/>
+<pinref part="TO-MAIN2" gate="1" pin="2"/>
 <wire x1="410.845" y1="9.8425" x2="405.765" y2="9.8425" width="0.1524" layer="91"/>
 <label x="405.765" y="9.8425" size="1.27" layer="95" rot="R180" xref="yes"/>
@@
 <wire x1="410.845" y1="12.3825" x2="403.225" y2="12.3825" width="0.1524" layer="91"/>
 <label x="403.225" y="12.3825" size="1.27" layer="95" rot="R180" xref="yes"/>
-<pinref part="TO-UI3" gate="1" pin="4"/>
+<pinref part="TO-MAIN2" gate="1" pin="4"/>
 </segment>
 <segment>
@@
 <segment>
 <pinref part="VDD4" gate="G$1" pin="VDD"/>
-<pinref part="TO-UI3" gate="1" pin="14"/>
+<pinref part="TO-MAIN2" gate="1" pin="14"/>
 <wire x1="407.4795" y1="30.4165" x2="407.4795" y2="25.0825" width="0.1524" layer="91"/>
 <wire x1="407.4795" y1="25.0825" x2="410.845" y2="25.0825" width="0.1524" layer="91"/>
@@
 <net name="N$13" class="0">
 <segment>
-<pinref part="TO-UI3" gate="1" pin="1"/>
+<pinref part="TO-MAIN2" gate="1" pin="1"/>
 <pinref part="USB-POLY" gate="G$1" pin="2"/>
 <wire x1="428.625" y1="9.8425" x2="426.085" y2="9.8425" width="0.1524" layer="91"/>

Commit message: #早く仕上げろー
Parts:
- added C1, C2: 0.1u, resistor:C-EUC1608
- added FT-R1, FT-R2, FT-R5: 330, 0@Mylibrary-main1:R-US_R0805
- added FT-R3, FT-R4: 27, 0@Mylibrary-main1:R-US_R0805
- added FT-R6: 100, 0@Mylibrary-main1:R-US_R0805
- added IC3: FT230XS, ftdichip:FT230XS
- added LED1, LED2, LED3: (no value), led:LEDCHIP-LED0805
- added SV1: (no value), 0con-lstb:MA05-1
- added U$2: USB-PAD, USB-PAD:USB-PAD
- added U$3: I-05318_ＮＳＳＷ１５７Ｔ, Akizuki:I-05318_ＮＳＳＷ１５７Ｔ
- added USB-POLY1: 350mA, polyswitch:PTC-F0805MP
- USB-POLY: value 100mA -> 400mA; device bel-fuse:0ZCH0200FF2E -> polyswitch:PTC-MF-5,1
Connections:
- new net +3V3-FT: C2.1, FT-R1.2, FT-R2.2, IC3.!RESET, IC3.3V3OUT, IC3.VCCIO, SV1.2
- new net GNDA: IC3.GND, LED3.C, U$2.GND, U$3.C
- new net N$19: FT-R2.1, LED2.A
- new net N$20: FT-R1.1, LED1.A
- new net N$22: FT-R3.2, U$2.D+
- new net N$23: FT-R3.1, IC3.USBDP
- new net N$24: FT-R4.1, IC3.USBDM
- new net N$25: FT-R4.2, U$2.D-
- new net N$26: C1.2, C2.2, IC3.GND@1, SV1.5
- new net N$27: U$2.VCC, USB-POLY1.2
- new net N$28: FT-R5.1, LED3.A
- new net N$29: FT-R6.1, U$3.A
- new net RXD: IC3.RXD, SV1.3
- new net RXLED: IC3.CBUS1, LED2.C
- new net TXD: IC3.TXD, SV1.4
- new net TXLED: IC3.CBUS2, LED1.C
- new net V+: C1.1, FT-R5.2, FT-R6.2, IC3.VCC, SV1.1, USB-POLY1.1
Other:
- note added: "UI"

Commit message: #update 大体完成　由利倫見れたら見てw
Parts:
- added CN1, CN13: (no value), jst-vh:B3P-VH
- added SJ1, SJ3: (no value), jumper:SJ2WW
- renumbered LED1 to TX-LED, LED2 to RX-LED
Connections:
- new net LED1: CN13.2, U$1.PB15
- new net LED2: CN1.2, U$1.PB14
- new net N$1: CN1.1, SJ1.2
- new net N$37: CN13.1, SJ3.2
- net +5V: now also SJ1.3, SJ3.3
- net +9V: now also SJ1.1, SJ3.1
- net GND: now also CN1.3, CN13.3

Commit message: #update ほぼ完成、F7,UI,KeyHolder基板ガーバ出力済み、main基板はあとはベタ確認とシルク最終チェック。明日の夜発注する！
Connections:
- net EMERGENCY: now also TO-MAIN.3; no longer TO-MAIN.2
- net GND: now also TO-MAIN.2; no longer TO-MAIN.1
Changed lines of the file:
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@@
 <part name="IC2" library="0linear-technology" deviceset="LTC485" device="N" package3d_urn="urn:adsk.eagle:package:16059/1"/>
 <part name="TO-MAIN" library="0con-harting-ml" deviceset="ML14" device=""/>
-<part name="GND44" library="supply1" deviceset="GND" device=""/>
 <part name="GND1" library="supply1" deviceset="GND" device=""/>
 <part name="S1" library="0switch" deviceset="255SB" device=""/>
@@
 <part name="GND12" library="supply1" deviceset="GND" device=""/>
 <part name="SUPPLY19" library="supply2" library_urn="urn:adsk.eagle:library:372" deviceset="+5V" device=""/>
+<part name="GND13" library="supply1" deviceset="GND" device=""/>
 </parts>
 <sheets>
@@
 <attribute name="NAME" x="151.13" y="23.622" size="1.778" layer="95"/>
 </instance>
-<instance part="GND44" gate="1" x="167.64" y="-7.62" smashed="yes">
-<attribute name="VALUE" x="165.1" y="-10.16" size="1.778" layer="96"/>
-</instance>
 <instance part="GND1" gate="1" x="38.1" y="68.58" smashed="yes">
 <attribute name="VALUE" x="35.56" y="66.04" size="1.778" layer="96"/>
@@
 <instance part="SUPPLY19" gate="+5V" x="193.04" y="119.38" smashed="yes">
 <attribute name="VALUE" x="191.135" y="122.555" size="1.778" layer="96"/>
+</instance>
+<instance part="GND13" gate="1" x="144.78" y="-5.08" smashed="yes">
+<attribute name="VALUE" x="142.24" y="-7.62" size="1.778" layer="96"/>
 </instance>
 </instances>
@@
 </net>
 <net name="GND" class="0">
-<segment>
-<pinref part="TO-MAIN" gate="1" pin="1"/>
-<wire x1="162.56" y1="5.08" x2="167.64" y2="5.08" width="0.1524" layer="91"/>
-<wire x1="167.64" y1="5.08" x2="167.64" y2="-5.08" width="0.1524" layer="91"/>
-<pinref part="GND44" gate="1" pin="GND"/>
-</segment>
 <segment>
 <pinref part="U$1" gate="G$1" pin="GND2"/>
@@
 <wire x1="177.8" y1="106.68" x2="177.8" y2="101.6" width="0.1524" layer="91"/>
 <pinref part="GND12" gate="1" pin="GND"/>
+</segment>
+<segment>
+<pinref part="GND13" gate="1" pin="GND"/>
+<pinref part="TO-MAIN" gate="1" pin="2"/>
+<wire x1="144.78" y1="-2.54" x2="144.78" y2="5.08" width="0.1524" layer="91"/>
+<wire x1="144.78" y1="5.08" x2="147.32" y2="5.08" width="0.1524" layer="91"/>
 </segment>
 </net>
@@
 <net name="EMERGENCY" class="0">
 <segment>
-<pinref part="TO-MAIN" gate="1" pin="2"/>
-<wire x1="147.32" y1="5.08" x2="142.24" y2="5.08" width="0.1524" layer="91"/>
-<label x="142.24" y="5.08" size="1.27" layer="95" rot="R180" xref="yes"/>
-</segment>
-<segment>
 <pinref part="U$1" gate="G$1" pin="PA4"/>
 <wire x1="60.96" y1="68.58" x2="58.42" y2="68.58" width="0.1524" layer="91"/>
 <label x="58.42" y="68.58" size="1.27" layer="95" rot="R180" xref="yes"/>
 </segment>
+<segment>
+<pinref part="TO-MAIN" gate="1" pin="3"/>
+<wire x1="162.56" y1="7.62" x2="167.64" y2="7.62" width="0.1524" layer="91"/>
+<label x="167.64" y="7.62" size="1.27" layer="95" xref="yes"/>
+</segment>
 </net>
