File: F7&UI&keyholder.brd (EAGLE design)
At the start: 100 x 100 mm, 27 parts, among them IC2 LTC485N, IC4 MCP2561-E_P

Commit message: #update
Parts:
- TO-UI: device 0con-harting-ml:ML10 -> 0con-harting-ml:ML14
Changed lines of the file:
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@@
 <attribute name="VALUE" x="40.9575" y="4.445" size="1.27" layer="27"/>
 </element>
-<element name="TO-UI" library="0con-harting-ml" package="ML10" value="" x="78.105" y="21.2725" smashed="yes" rot="R270">
+<element name="TO-UI" library="0con-harting-ml" package="ML14" value="" x="78.105" y="21.2725" smashed="yes" rot="R270">
 <attribute name="MF" value="" x="78.105" y="21.2725" size="1.778" layer="27" rot="R270" display="off"/>
 <attribute name="MPN" value="" x="78.105" y="21.2725" size="1.778" layer="27" rot="R270" display="off"/>
@@
 <contactref element="BOOT0-STM" pad="3"/>
 <wire x1="86.92" y1="19.975" x2="93.42" y2="19.975" width="0" layer="19" extent="1-1"/>
-<wire x1="79.375" y1="23.8125" x2="86.92" y2="19.975" width="0" layer="19" extent="1-1"/>
+<wire x1="79.375" y1="26.3525" x2="86.92" y2="19.975" width="0" layer="19" extent="1-1"/>
 <wire x1="75.6675" y1="6.6675" x2="86.92" y2="19.975" width="0" layer="19" extent="1-1"/>
 </signal>
@@
 <contactref element="TO-UI" pad="6"/>
 <contactref element="ST-LINKV2" pad="4"/>
-<wire x1="63.5" y1="18.0975" x2="79.375" y2="21.2725" width="0" layer="19" extent="1-1"/>
+<wire x1="63.5" y1="18.0975" x2="79.375" y2="23.8125" width="0" layer="19" extent="1-1"/>
 </signal>
 <signal name="SWCLK">
 <contactref element="TO-UI" pad="7"/>
 <contactref element="ST-LINKV2" pad="2"/>
-<wire x1="63.5" y1="13.0175" x2="76.835" y2="18.7325" width="0" layer="19" extent="1-1"/>
+<wire x1="63.5" y1="13.0175" x2="76.835" y2="21.2725" width="0" layer="19" extent="1-1"/>
 </signal>
 <signal name="NRST">
@@
 <wire x1="86.285" y1="12.0375" x2="92.785" y2="12.0375" width="0" layer="19" extent="1-1"/>
 <wire x1="75.985" y1="9.2075" x2="86.285" y2="12.0375" width="0" layer="19" extent="1-1"/>
-<wire x1="76.835" y1="21.2725" x2="75.985" y2="9.2075" width="0" layer="19" extent="1-1"/>
-<wire x1="63.5" y1="20.6375" x2="76.835" y2="21.2725" width="0" layer="19" extent="1-1"/>
+<wire x1="76.835" y1="23.8125" x2="75.985" y2="9.2075" width="0" layer="19" extent="1-1"/>
+<wire x1="63.5" y1="20.6375" x2="76.835" y2="23.8125" width="0" layer="19" extent="1-1"/>
 </signal>
 <signal name="N$7">
@@
 <contactref element="RESET-STM" pad="1"/>
 <contactref element="RESET-STM" pad="2"/>
-<wire x1="76.835" y1="26.3525" x2="84.4525" y2="33.9725" width="0" layer="19" extent="1-1"/>
-<wire x1="66.995" y1="32.7025" x2="76.835" y2="26.3525" width="0" layer="19" extent="1-1"/>
-<wire x1="86.285" y1="16.5375" x2="76.835" y2="26.3525" width="0" layer="19" extent="1-1"/>
+<wire x1="76.835" y1="28.8925" x2="84.4525" y2="33.9725" width="0" layer="19" extent="1-1"/>
+<wire x1="66.995" y1="32.7025" x2="76.835" y2="28.8925" width="0" layer="19" extent="1-1"/>
+<wire x1="86.285" y1="16.5375" x2="76.835" y2="28.8925" width="0" layer="19" extent="1-1"/>
 <wire x1="92.785" y1="16.5375" x2="86.285" y2="16.5375" width="0" layer="19" extent="1-1"/>
 <wire x1="77.3675" y1="6.6675" x2="86.285" y2="16.5375" width="0" layer="19" extent="1-1"/>
@@
 <contactref element="TO-UI" pad="10"/>
 <contactref element="LED-5V" pad="A"/>
-<wire x1="79.375" y1="16.1925" x2="72.0725" y2="42.2275" width="0" layer="19" extent="1-1"/>
+<wire x1="79.375" y1="18.7325" x2="72.0725" y2="42.2275" width="0" layer="19" extent="1-1"/>
 </signal>
 <signal name="VCC/2">
@@
 <wire x1="86.92" y1="24.475" x2="78.4225" y2="38.735" width="0" layer="19" extent="1-1"/>
 <wire x1="93.42" y1="24.475" x2="86.92" y2="24.475" width="0" layer="19" extent="1-1"/>
-<wire x1="76.835" y1="16.1925" x2="86.92" y2="24.475" width="0" layer="19" extent="1-1"/>
-<wire x1="77.685" y1="9.2075" x2="76.835" y2="16.1925" width="0" layer="19" extent="1-1"/>
+<wire x1="76.835" y1="18.7325" x2="86.92" y2="24.475" width="0" layer="19" extent="1-1"/>
+<wire x1="77.685" y1="9.2075" x2="76.835" y2="18.7325" width="0" layer="19" extent="1-1"/>
 <wire x1="63.5" y1="10.4775" x2="77.685" y2="9.2075" width="0" layer="19" extent="1-1"/>
 </signal>

Commit message: #OTL 意外とやること多い
Parts:
- removed BOOT0-STM, RESET-STM: DTS-6, forprint:DTS-6
- removed LED-3V3, LED-5V: (no value), adafruit:LED5MM
- removed R1, R2: (no value), resistor:M0805
- removed TO-UI: (no value), 0con-harting-ml:ML14
- added CON1, CON2: XH-3, 0@Mylibrary-main1:CON3
- added J1, J2, J3, J4, J5, J6: XH-2, 0@Mylibrary-main1:CON2
- added Q1, Q2: BSS123, transistor-small-signal:SOT23
- added R3, R4: 4.7k, resistor:M0805
- added S3: (no value), switch-omron:B3F-40XX
- added SW1: (no value), special:EDG-03
- added TO-UI2: (no value), 0con-harting-ml:ML14
- moved S2 126.3 mm to (91.7, 85.9), turned to 180 degrees
- moved STM-R1 92.6 mm to (138.7, -59.7)
- moved STM-R2 92.6 mm to (138.4, -62.2)
- moved ST-LINKV2 18.5 mm to (56.4, 33.9)
Connections:
- removed net +5V/2: LED-5V.A, TO-UI.10
- removed net N$7: LED-5V.K, R1.2
- removed net N$8: LED-3V3.K, R2.1
- new net +12VS: TO-UI2.6
- new net +3V3S: SW1.2, TO-UI2.12
- new net 12V-SW: TO-UI2.3
- new net LIPO2: J1.P$1, TO-UI2.1
- new net MOTOR-FET: J2.P$1, TO-UI2.2
- new net N$2: Q1.1, R4.2
- new net N$3: Q2.1, R3.2
- new net N$6: J6.P$1, SW1.4, SW1.5, SW1.6
- new net VDD: J3.P$1, SW1.3, TO-UI2.14
- net +5VS: now also SW1.1, TO-UI2.7; no longer TO-UI.8
- net 3V3-SW: now also Q1.3, TO-UI2.4; no longer TO-UI.2
- net 5V-SW: now also Q2.3, TO-UI2.5; no longer TO-UI.3
- net BOOT0: now also S3.1, S3.2, TO-UI2.8; no longer BOOT0-STM.3, BOOT0-STM.4, TO-UI.4
- net GND2: now also J1.P$2, J2.P$2, J3.P$2, J6.P$2, Q1.2, Q2.2, R3.1, R4.1, S2.3, S2.4, TO-UI2.13; no longer R1.1, R2.2, RESET-STM.1, RESET-STM.2, TO-UI.1
- net NRST: now also S2.1, S2.2, TO-UI2.9; no longer RESET-STM.3, RESET-STM.4, TO-UI.5
- net SWCLK: now also TO-UI2.11; no longer TO-UI.7
- net SWDIO: now also TO-UI2.10; no longer TO-UI.6
- net VCC/2: now also S3.3, S3.4; no longer BOOT0-STM.1, BOOT0-STM.2, LED-3V3.A, TO-UI.9
Other:
- outline, holes or cut-outs redrawn

Commit message: #update UI,F7 だいたい完成 #todo シルク
Parts:
- removed CON1, CON2: XH-3, 0@Mylibrary-main1:CON3
- removed J1, J2, J3, J4, J5, J6: XH-2, 0@Mylibrary-main1:CON2
- removed Q1, Q2: BSS123, transistor-small-signal:SOT23
- removed S2: (no value), switch-omron:B3F-40XX
- removed TO-UI2: (no value), 0con-harting-ml:ML14
- added 12V-FET, 3V3-FET, 5V-FET: BSS123, transistor-small-signal:SOT23
- added 12V-KEY, 12V-LED, LIPO-LED, MOTOR-KEY, MOTOR-LED, VOLTAGE: XH-2, 0@Mylibrary-main1:CON2
- added 3V3-SW, 5V-SW: XH-3, 0@Mylibrary-main1:CON3
- added LED-R1, LED-R2, LED-R3: ?, resistor:M0805
- added R1: 4.7k, resistor:M0805
- added R2, R5, R6: 1k, resistor:M0805
- added S4: ST12-303FCG, ST12-303FCG:ST12303FCG
- added SW-R1, SW-R2: 330, 0@Mylibrary-main1:R0805
- added TO-UI3: (no value), 0con-harting-ml:ML14
- added USB-POLY: 100mA, bel-fuse:0ZCH
- S3: value (none) -> ST12-303FCG; device switch-omron:B3F-40XX -> ST12-303FCG:ST12303FCG
- SW1: device special:EDG-03 -> 0special:EDG-03
- moved SW1 192.1 mm to (60.0, 48.5), turned to 270 degrees
- moved R4 182.8 mm to (61.0, 84.0), flipped to the bottom, turned to 90 degrees
- moved R3 164.0 mm to (61.0, 69.0), flipped to the bottom, turned to 90 degrees
- moved STM-R1 145.0 mm to (98.1, 79.4), flipped to the bottom, turned to 270 degrees
- moved STM-R2 133.1 mm to (98.1, 64.7), flipped to the bottom, turned to 270 degrees
- moved S3 1.13 mm to (91.8, 70.9)
- moved RS485-S 0.64 mm to (13.3, 37.5), turned to 90 degrees
Connections:
- removed net VCC/2: S3.3, S3.4, ST-LINKV2.1, STM-R1.2
- new net N$10: 5V-SW.P$1, R5.2
- new net N$11: S4.ANODE, SW-R1.2
- new net N$12: S3.ANODE, SW-R2.2
- new net N$13: TO-UI3.1, USB-POLY.2
- new net N$14: LED-R1.2, LIPO-LED.P$1
- new net N$15: LED-R2.2, MOTOR-LED.P$1
- new net N$16: 12V-LED.P$1, LED-R3.2
- new net N$7: 12V-FET.1, R1.2, R6.1
- new net N$8: 12V-KEY.P$2, R6.2
- new net N$9: 3V3-SW.P$1, R2.2
- net +12VS: now also TO-UI3.3; no longer TO-UI2.6
- net +3V3S: now also S3.3, S3.4, ST-LINKV2.1, STM-R1.2, SW-R1.1, SW-R2.1, TO-UI3.12; no longer TO-UI2.12
- net +5VS: now also TO-UI3.7; no longer TO-UI2.7
- net 12V-SW: now also 12V-FET.3, TO-UI3.4; no longer TO-UI2.3
- net 3V3-SW: now also 3V3-FET.3, TO-UI3.6; no longer Q1.3, TO-UI2.4
- net 5V-SW: now also 5V-FET.3, TO-UI3.5; no longer Q2.3, TO-UI2.5
- net BOOT0: now also TO-UI3.8; no longer TO-UI2.8
- net F7-F4-SIG1: now also U$1.PC8; no longer U$1.PJ0
- net F7-F4-SIG2: now also U$1.PJ0; no longer U$1.PC8
- net F7-RS-SIG1: now also U$1.PJ3; no longer U$1.PF7
- net F7-RS-SIG2: now also U$1.PF7; no longer U$1.PJ3
- net GND2: now also 12V-FET.2, 12V-LED.P$2, 3V3-FET.2, 3V3-SW.P$3, 5V-FET.2, 5V-SW.P$3, LIPO-LED.P$2, MOTOR-LED.P$2, R1.1, S3.CATHODE, S4.3, S4.4, S4.CATHODE, TO-UI3.13, VOLTAGE.P$2; no longer J1.P$2, J2.P$2, J3.P$2, J6.P$2, Q1.2, Q2.2, S2.3, S2.4, TO-UI2.13
- net LIPO2: now also LED-R1.1, MOTOR-KEY.P$1, USB-POLY.1; no longer J1.P$1, TO-UI2.1
- net MOTOR-FET: now also LED-R2.1, MOTOR-KEY.P$2, TO-UI3.2; no longer J2.P$1, TO-UI2.2
- net N$2: now also 3V3-FET.1, R2.1; no longer Q1.1
- net N$3: now also 5V-FET.1, R5.1; no longer Q2.1
- net N$6: now also VOLTAGE.P$1; no longer J6.P$1
- net NRST: now also S4.1, S4.2, TO-UI3.9; no longer S2.1, S2.2, TO-UI2.9
- net SWCLK: now also TO-UI3.10; no longer TO-UI2.11
- net SWDIO: now also TO-UI3.11; no longer TO-UI2.10
- net VDD: now also 12V-KEY.P$1, 3V3-SW.P$2, 5V-SW.P$2, LED-R3.1, TO-UI3.14; no longer J3.P$1, TO-UI2.14
Routing:
- net VDD: track 0.00 -> 134.0 mm
- net +3V3S: track 0.00 -> 116.0 mm
- net NRST: track 0.00 -> 86.6 mm
- net LIPO2: track 0.00 -> 79.3 mm, vias 0 -> 1
- net 12V-SW: track 0.00 -> 67.7 mm, vias 0 -> 1
- net +9V: track 0.00 -> 63.1 mm
- net N$6: track 0.00 -> 57.9 mm
- net MOTOR-FET: track 0.00 -> 44.2 mm
- net BOOT0: track 0.00 -> 37.9 mm
- net SWCLK: track 0.00 -> 34.1 mm
- net 3V3-SW: track 0.00 -> 29.6 mm, vias 0 -> 1
- net F7-RS-SIG2: track 0.00 -> 28.5 mm
- net F7-RS-SIG1: track 0.00 -> 27.5 mm
- net RS-CHB: track 0.00 -> 26.9 mm
- net SWDIO: track 0.00 -> 25.4 mm
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- added copper zone on layer 1, net GND2
- removed copper zone on layer 1, net GND
- removed copper zone on layer 16, net GND
Other:
- outline, holes or cut-outs redrawn

Commit message: #update UI,F7 シルク官僚
Parts:
- IC2: device linear-technology:DIL08 -> 0linear-technology:DIL08
- moved BUZ-R1 23.6 mm to (32.7, 6.67)
- moved SG1 6.02 mm to (40.6, 32.4)
- moved LIPO-LED 1.40 mm to (56.7, 11.8), turned to 270 degrees
- renumbered TO-F7 to TO-MAIN, TO-UI3 to TO-MAIN2
Routing:
- net VCC: track 0.00 -> 63.4 mm, vias 0 -> 1
- net USART6-TX: track 0.00 -> 55.4 mm
- net RS-SIG: track 0.00 -> 45.6 mm, vias 0 -> 1
- net USART6-RX: track 0.00 -> 44.7 mm
- net CAN1-RX: track 0.00 -> 35.9 mm
- net +5V: track 0.00 -> 35.5 mm
- net CAN1-TX: track 0.00 -> 34.1 mm
- net BUZZER1: track 0.00 -> 28.1 mm, vias 0 -> 1
- net F7-F4-SIG2: track 0.00 -> 23.9 mm
- net F7-F4-SIG1: track 0.00 -> 22.9 mm
- net HUMAN1: track 0.00 -> 22.9 mm
- net EMERGENCY: track 0.00 -> 19.3 mm
- net +9V: track 63.1 -> 50.0 mm
- net GND: track 0.00 -> 6.89 mm, vias 0 -> 208
- net +3V3S: track 116.0 -> 117.8 mm
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- added copper zone on layer 1, net GND
- added copper zone on layer 16, net GND
Other:
- board text added: "G"

Commit message: #早く仕上げろー
Parts:
- added C1, C2: 0.1u, resistor:C1608
- added FT-R1, FT-R2, FT-R5: 330, 0@Mylibrary-main1:R0805
- added FT-R3, FT-R4: 27, 0@Mylibrary-main1:R0805
- added FT-R6: 100, 0@Mylibrary-main1:R0805
- added IC3: FT230XS, ftdichip:SSOP16
- added LED1, LED2, LED3: (no value), led:CHIP-LED0805
- added SV1: (no value), 0con-lstb:MA05-1
- added U$2: USB-PAD, USB-PAD:USB
- added U$3: I-05318_ＮＳＳＷ１５７Ｔ, Akizuki:NSSW157T
- added U$5: (no value), Carrot:CARROT
- added U$6: (no value), Carrot:DDPROJECT2-TOP
- added USB-POLY1: 350mA, polyswitch:F0805MP
- USB-POLY: value 100mA -> 400mA; device bel-fuse:0ZCH -> polyswitch:MF-5/1
- moved USB-POLY 9.26 mm to (81.0, 50.2), flipped to the bottom, turned to 40 degrees
Connections:
- new net +3V3-FT: C2.1, FT-R1.2, FT-R2.2, IC3.10, IC3.11, IC3.3, SV1.2
- new net GNDA: IC3.5, LED3.C, U$2.GND, U$3.CATHODE
- new net N$19: FT-R2.1, LED2.A
- new net N$20: FT-R1.1, LED1.A
- new net N$22: FT-R3.2, U$2.D+
- new net N$23: FT-R3.1, IC3.8
- new net N$24: FT-R4.1, IC3.9
- new net N$25: FT-R4.2, U$2.D-
- new net N$26: C1.2, C2.2, IC3.13, SV1.5
- new net N$27: U$2.VCC, USB-POLY1.2
- new net N$28: FT-R5.1, LED3.A
- new net N$29: FT-R6.1, U$3.ANODE
- new net RXD: IC3.4, SV1.3
- new net RXLED: IC3.14, LED2.C
- new net TXD: IC3.1, SV1.4
- new net TXLED: IC3.7, LED1.C
- new net V+: C1.1, FT-R5.2, FT-R6.2, IC3.12, SV1.1, USB-POLY1.1
Routing:
- net +3V3-FT: track 0.00 -> 48.5 mm, vias 0 -> 2
- net V+: track 0.00 -> 47.2 mm
- net N$26: track 0.00 -> 36.3 mm, vias 0 -> 2
- net RXD: track 0.00 -> 31.7 mm, vias 0 -> 2
- net TXD: track 0.00 -> 29.0 mm, vias 0 -> 2
- net TXLED: track 0.00 -> 13.6 mm
- net RXLED: track 0.00 -> 9.62 mm
- net N$27: track 0.00 -> 8.27 mm
- net N$13: track 1.77 -> 9.59 mm
- net N$25: track 0.00 -> 7.73 mm
- net N$22: track 0.00 -> 7.73 mm
- net N$23: track 0.00 -> 5.01 mm
- net N$24: track 0.00 -> 4.46 mm
- net N$28: track 0.00 -> 2.55 mm
- net N$20: track 0.00 -> 1.91 mm
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- added copper zone on layer 1, net GNDA
Other:
- outline, holes or cut-outs redrawn

Commit message: #update 大体完成　由利倫見れたら見てw
Parts:
- added CN1, CN13: (no value), jst-vh:B3P-VH
- added SJ1, SJ3: (no value), jumper:SJ_2W
- renumbered LED1 to TX-LED, LED2 to RX-LED
Connections:
- new net LED1: CN13.2, U$1.PB15
- new net LED2: CN1.2, U$1.PB14
- new net N$1: CN1.1, SJ1.2
- new net N$37: CN13.1, SJ3.2
- net +5V: now also SJ1.3, SJ3.3
- net +9V: now also SJ1.1, SJ3.1
- net GND: now also CN1.3, CN13.3
Routing:
- net +5V: track 35.5 -> 77.3 mm
- net +9V: track 50.0 -> 74.4 mm, vias 0 -> 3
- net GNDA: track 0.00 -> 20.3 mm, vias 0 -> 9
- net LED1: track 0.00 -> 13.7 mm
- net N$37: track 0.00 -> 12.9 mm
- net N$1: track 0.00 -> 12.9 mm, vias 0 -> 1
- net LED2: track 0.00 -> 11.8 mm
- net CAN1-RX: track 35.9 -> 39.2 mm
- net CAN1-TX: track 34.1 -> 37.2 mm
- net GND: vias 208 -> 168
- net BUZZER1: vias 1 -> 3
Other:
- board text added: "+3V3"
- board text added: "+5V"
- board text added: "GND"
- board text added: "RXD"
- board text added: "TXD"
