File: mainboard.brd (EAGLE design)
At the start: 144.9 x 134.8 mm, 155 parts, among them CON1 XH-3, IC1 STM32F429VGT, IC2 LTC485N, IC3 DP83848, IC4 MCP2561-E_P, Q2 IRF9530, Q3 IRF9530, Q4 IRF9530, Q5 IRF9530, X1 RASPI_BOARD_B+#_FP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

Commit message: #OTL 意外とやること多い
Parts:
- removed SUPPLY9: MAIN, con-ptr500:AK500/2
- removed TO-UI: (no value), 0con-harting-ml:ML14
- added TO-UI3: (no value), 0con-harting-ml:ML14
- added U$2: XT60, XT60:XT60
- CN11: device jst-vh:B2P-VH -> jst-vh:B3P-VH
- moved GND-CH 76.8 mm to (15.0, 82.4)
- moved RESET-STM 11.7 mm to (40.9, 19.1)
- moved STM-R1 11.5 mm to (43.2, 25.1)
- moved BOOT0-STM 11.4 mm to (48.3, 19.1)
Connections:
- removed net N$38: Q3.D, SUPPLY9.1, X2.1
- removed net N$40: MAINSW2.1, Q5.G, SP-R6.1, SUOPPLY-SW2.P$1
- removed net N$5: Q3.S, Q5.S, SP-R6.2
- new net +12VS: Q3.S, Q5.S, SP-R6.2, TO-UI3.6
- new net 12V-B: Q3.D, U$2.+, X2.1
- new net 12V-SW: MAINSW2.1, Q5.G, SP-R6.1, SUOPPLY-SW2.P$1, TO-UI3.3
- new net LIPO2: TO-UI3.1
- new net MOTOR-FET: CN11.3, TO-UI3.2
- net +3V3: no longer TO-UI.13
- net +3V3S: now also TO-UI3.12; no longer TO-UI.9
- net +5V: no longer TO-UI.14
- net +5VS: now also TO-UI3.7; no longer TO-UI.8
- net +9V: now also TO-UI3.14; no longer TO-UI.12
- net 3V3-SW: now also TO-UI3.4; no longer TO-UI.2
- net 5V-SW: now also TO-UI3.5; no longer TO-UI.3
- net BOOT0: now also TO-UI3.8; no longer TO-UI.4
- net GND: now also TO-UI3.13, U$2.-; no longer SUPPLY9.2, TO-UI.1
- net NRST: now also TO-UI3.9; no longer TO-UI.5
- net SWCLK: now also TO-UI3.11; no longer TO-UI.7
- net SWDIO: now also TO-UI3.10; no longer TO-UI.6
Routing:
- net +3V3S: track 42.8 -> 145.8 mm, vias 0 -> 4
- net +12VS: track 0.00 -> 91.3 mm
- net 12V-SW: track 0.00 -> 85.1 mm
- net 12V-B: track 0.00 -> 47.0 mm
- net LIPO: track 76.2 -> 115.6 mm
- net MOTOR-FET: track 0.00 -> 31.4 mm
- net SWDIO: track 101.0 -> 129.6 mm
- net SWCLK: track 88.5 -> 115.1 mm
- net N$38: track 25.0 -> 0.00 mm
- net +5V: track 143.6 -> 168.0 mm, vias 1 -> 2
- net N$40: track 22.8 -> 0.00 mm
- net NRST: track 140.4 -> 157.4 mm, vias 4 -> 3
- net GND: track 153.2 -> 168.4 mm
- net N$5: track 9.31 -> 0.00 mm
- net +3V3: track 647.3 -> 655.6 mm, vias 27 -> 26
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- added copper zone on layer 1, net 12V-B

Commit message: #update UI,F7 だいたい完成 #todo シルク
Parts:
- USB-POLY: value 350mA -> 100mA
- moved TO-UI3 53.3 mm to (31.0, 41.7), turned to 90 degrees
Connections:
- removed net +9V: TO-UI3.14
- removed net LIPO2: TO-UI3.1
- net +12V: now also TO-UI3.14
- net +12VS: now also TO-UI3.3; no longer TO-UI3.6
- net 12V-SW: now also TO-UI3.4; no longer TO-UI3.3
- net 3V3-SW: now also TO-UI3.6; no longer TO-UI3.4
- net LIPO: now also TO-UI3.1
- net SWCLK: now also TO-UI3.10; no longer TO-UI3.11
- net SWDIO: now also TO-UI3.11; no longer TO-UI3.10
Routing:
- net SWDIO: track 129.6 -> 97.3 mm
- net SWCLK: track 115.1 -> 90.4 mm
- net +5V: track 168.0 -> 191.4 mm, vias 2 -> 4
- net +3V3S: track 145.8 -> 125.4 mm, vias 4 -> 1
- net BOOT0: track 108.1 -> 120.0 mm
- net +12VS: track 91.3 -> 99.2 mm
- net +3V3: track 655.6 -> 661.5 mm
- net +5VS: track 359.7 -> 364.2 mm
- net GND: track 168.4 -> 172.5 mm
- net 5V-SW: track 68.8 -> 72.8 mm
- net NRST: track 157.4 -> 155.6 mm, vias 3 -> 4
- net FET1: track 91.9 -> 92.9 mm
- net LIPO: track 115.6 -> 114.7 mm
- net FET2: track 89.2 -> 90.0 mm
- net +12V: track 244.4 -> 245.0 mm, vias 8 -> 7

Commit message: #早く仕上げろー
Parts:
- removed CN10: (no value), jst-vh:B2P-VH
- removed FET-R1, FET-R2, FET-R3, FET-R4: 100, 0@Mylibrary-main1:R0805
- removed FETR1: 4.7k, resistor-dil:EXBN8V
- removed SP-LED: (no value), led:CHIPLED_0805
- removed SP-R9: 330, 0@Mylibrary-main1:R0805
- removed T1, T2: (no value), zetex:SO8
- added 100, SP-R5: 330, 0@Mylibrary-main1:R0805
- added SP-LED1, SP-LED2: (no value), led:CHIPLED_0805
- added X4, X5, X6: (no value), con-ptr500:AK500/2
- USB-POLY: value 100mA -> 400mA; device bel-fuse:0ZCH -> polyswitch:F0805MP
- moved CN11 27.2 mm to (50.0, 5.08)
- moved JP1 19.6 mm to (57.0, 25.8), turned to 270 degrees
Connections:
- removed net N$17: SP-LED.C, SP-R9.2
- removed net N$29: FET-R1.1, FETR1.8, T1.2
- removed net N$30: FET-R2.1, FETR1.7, T1.4
- removed net N$32: FET-R4.1, FETR1.5, T2.4
- removed net N$33: FET-R3.1, FETR1.6, T2.2
- new net N$24: 100.2, SP-LED2.C
- new net N$5: SP-LED1.C, SP-R5.2
- net +12V: now also X6.1
- net +3V3: now also SP-LED2.A, X5.1
- net +5V: now also SP-LED1.A, X4.1
- net +5VS: no longer SP-LED.A
- net FET1: no longer FET-R1.2
- net FET2: no longer FET-R2.2
- net FET3: no longer FET-R3.2
- net FET4: no longer FET-R4.2
- net GND: now also 100.1, SP-R5.1, X4.2, X5.2, X6.2; no longer CN10.2, FETR1.1, FETR1.2, FETR1.3, FETR1.4, SP-R9.1, T1.1, T1.3, T2.1, T2.3
- net LED1: no longer T1.7, T1.8
- net LED2: no longer T1.5, T1.6
- net LED3: no longer T2.7, T2.8
- net LED4: no longer T2.5, T2.6
- net LIPO: no longer CN10.1
Routing:
- net LIPO: track 114.7 -> 55.9 mm
- net MOTOR-FET: track 31.6 -> 8.10 mm
- net +12V: track 245.0 -> 265.3 mm
- net +5V: track 191.4 -> 209.6 mm
- net N$32: track 14.9 -> 0.00 mm, vias 2 -> 0
- net N$33: track 12.9 -> 0.00 mm
- net +5VS: track 364.2 -> 352.2 mm
- net N$29: track 11.9 -> 0.00 mm, vias 2 -> 0
- net N$30: track 10.1 -> 0.00 mm
- net LED4: track 9.32 -> 6.37 mm
- net LED2: track 9.32 -> 6.37 mm
- net FET2: track 90.0 -> 87.1 mm
- net FET3: track 79.7 -> 77.0 mm
- net FET1: track 92.9 -> 90.5 mm
- net N$17: track 2.31 -> 0.00 mm
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
Commit message: #update 大体完成　由利倫見れたら見てw
Parts:
- removed CN2, CN3, CN4, CN5: (no value), jst-vh:B2P-VH
- added LED1, LED2, LED3, LED4: (no value), jst-vh:B3P-VH
- added SJ1, SJ2, SJ3, SJ4: (no value), jumper:SJ_2W
- renumbered CN11 to LIPO, CN6 to LED5, CN7 to LED6, CN8 to LED8, CN9 to LED7, CON1 to PING
Connections:
- removed net LED1: CN2.2
- removed net LED2: CN3.2
- removed net LED3: CN5.2
- removed net LED4: CN4.2
- new net N$17: LED3.1, SJ1.2
- new net N$32: LED1.1, SJ2.2
- new net N$37: LED4.1, SJ3.2
- new net N$40: LED2.1, SJ4.2
- net +12V: now also SJ1.1, SJ2.1, SJ3.1, SJ4.1; no longer CN2.1, CN3.1, CN4.1, CN5.1
- net +5V: now also SJ1.3, SJ2.3, SJ3.3, SJ4.3
- net FET1: now also LED1.2
- net FET2: now also LED2.2
- net FET3: now also LED3.2
- net FET4: now also LED4.2
- net GND: now also LED1.3, LED2.3, LED3.3, LED4.3
Routing:
- net MOTOR-FET: track 8.10 -> 45.4 mm, vias 0 -> 1
- net LIPO: track 55.9 -> 86.7 mm, vias 2 -> 3
- net +5V: track 209.6 -> 235.4 mm, vias 4 -> 0
- net FET4: track 74.1 -> 96.7 mm, vias 4 -> 5
- net FET2: track 87.1 -> 108.0 mm, vias 4 -> 3
- net +3V3: track 661.4 -> 681.1 mm
- net +5VS: track 352.2 -> 337.4 mm
- net +12V: track 265.3 -> 277.4 mm, vias 7 -> 10
- net FET3: track 77.0 -> 86.7 mm, vias 4 -> 5
- net LED1: track 9.11 -> 0.00 mm
- net LED3: track 8.85 -> 0.00 mm
- net FET1: track 90.5 -> 97.6 mm, vias 4 -> 3
- net LED4: track 6.37 -> 0.00 mm
- net LED2: track 6.37 -> 0.00 mm
- net N$37: track 0.00 -> 4.93 mm
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Other:
- board text added: "+12V"
- board text added: "+3V3"
- board text added: "+5V"
- board text added: "ADC"
- board text added: "BOOT0"
- board text added: "E"
- board text added: "G"
- board text added: "GND"
- board text added: "MAX DC +25V"
- board text added: "NRST"
- board text added: "RESET"
- board text added: "S"
- board text added: "SIG"
- board text added: "SWCLK"
- board text added: "SWDIO"
