File: mainboard.sch (EAGLE design)
At the start: 155 parts, among them CON1 XH-3, IC1 STM32F429VGT, IC2 LTC485N, IC3 DP83848, IC4 MCP2561-E_P, Q2 IRF9530, Q3 IRF9530, Q4 IRF9530, Q5 IRF9530, X1 RASPI_BOARD_B+#_FP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

Commit message: #OTL 意外とやること多い
Parts:
- removed SUPPLY9: MAIN, con-ptr500:AK500/2
- removed TO-UI: (no value), 0con-harting-ml:ML14
- added TO-UI3: (no value), 0con-harting-ml:ML14
- added U$2: XT60, XT60:XT60
- CN11: device jst-vh:B2P-VH -> jst-vh:B3P-VH
Connections:
- removed net N$38: Q3.D, SUPPLY9-1.KL, X2.1
- removed net N$40: MAINSW2.1, Q5.G, SP-R6.1, SUOPPLY-SW2.1
- removed net N$5: Q3.S, Q5.S, SP-R6.2
- new net +12VS: Q3.S, Q5.S, SP-R6.2, TO-UI3.6
- new net 12V-B: Q3.D, U$2.VCC, X2.1
- new net 12V-SW: MAINSW2.1, Q5.G, SP-R6.1, SUOPPLY-SW2.1, TO-UI3.3
- new net LIPO2: TO-UI3.1
- new net MOTOR-FET: CN11.3, TO-UI3.2
- net +3V3: no longer TO-UI.13
- net +3V3S: now also TO-UI3.12; no longer TO-UI.9
- net +5V: no longer TO-UI.14
- net +5VS: now also TO-UI3.7; no longer TO-UI.8
- net +9V: now also TO-UI3.14; no longer TO-UI.12
- net 3V3-SW: now also TO-UI3.4; no longer TO-UI.2
- net 5V-SW: now also TO-UI3.5; no longer TO-UI.3
- net BOOT0: now also TO-UI3.8; no longer TO-UI.4
- net GND: now also TO-UI3.13, U$2.GND; no longer SUPPLY9-2.KL, TO-UI.1
- net NRST: now also TO-UI3.9; no longer TO-UI.5
- net SWCLK: now also TO-UI3.11; no longer TO-UI.7
- net SWDIO: now also TO-UI3.10; no longer TO-UI.6

Commit message: #update UI,F7 だいたい完成 #todo シルク
Parts:
- USB-POLY: value 350mA -> 100mA
Connections:
- removed net +9V: TO-UI3.14
- removed net LIPO2: TO-UI3.1
- net +12V: now also TO-UI3.14
- net +12VS: now also TO-UI3.3; no longer TO-UI3.6
- net 12V-SW: now also TO-UI3.4; no longer TO-UI3.3
- net 3V3-SW: now also TO-UI3.6; no longer TO-UI3.4
- net LIPO: now also TO-UI3.1
- net SWCLK: now also TO-UI3.10; no longer TO-UI3.11
- net SWDIO: now also TO-UI3.11; no longer TO-UI3.10
Changed lines of the file:
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@@
 <part name="+3V18" library="supply1" deviceset="+3V3" device=""/>
 <part name="X3" library="Akizuki" deviceset="C-07674_USB-A" device=""/>
-<part name="USB-POLY" library="bel-fuse" deviceset="0ZCH*" device="" technology="0200FF2E" value="350mA"/>
+<part name="USB-POLY" library="bel-fuse" deviceset="0ZCH*" device="" technology="0200FF2E" value="100mA"/>
 <part name="GND41" library="0@Mylibrary-main1" deviceset="GND" device=""/>
 <part name="CN2" library="jst-vh" deviceset="B2P-VH" device=""/>
@@
 <wire x1="5.08" y1="-147.32" x2="5.08" y2="-139.7" width="0.1524" layer="91"/>
 <pinref part="SUPPLY5" gate="G$1" pin="+9V"/>
+<label x="40.64" y="-134.62" size="1.778" layer="95"/>
+</segment>
+<segment>
+<pinref part="SUPPLY7" gate="G$1" pin="+9V"/>
+<pinref part="TO-UI3" gate="1" pin="14"/>
+<wire x1="-9.144" y1="-188.468" x2="-9.144" y2="-193.3575" width="0.1524" layer="91"/>
+<wire x1="-9.144" y1="-193.3575" x2="-5.715" y2="-193.3575" width="0.1524" layer="91"/>
 </segment>
 </net>
@@
 </segment>
 <segment>
-<wire x1="-5.715" y1="-206.0575" x2="-13.335" y2="-206.0575" width="0.1524" layer="91"/>
-<label x="-13.335" y="-206.0575" size="1.27" layer="95" rot="R180" xref="yes"/>
-<pinref part="TO-UI3" gate="1" pin="4"/>
+<pinref part="TO-UI3" gate="1" pin="6"/>
+<wire x1="-5.715" y1="-203.5175" x2="-10.795" y2="-203.5175" width="0.1524" layer="91"/>
+<label x="-10.795" y="-203.5175" size="1.27" layer="95" rot="R180" xref="yes"/>
 </segment>
 </net>
@@
 </segment>
 <segment>
-<wire x1="-5.715" y1="-198.4375" x2="-10.795" y2="-198.4375" width="0.1524" layer="91"/>
-<label x="-10.795" y="-198.4375" size="1.27" layer="95" rot="R180" xref="yes"/>
-<pinref part="TO-UI3" gate="1" pin="10"/>
+<wire x1="9.525" y1="-195.8975" x2="17.145" y2="-195.8975" width="0.1524" layer="91"/>
+<label x="17.145" y="-195.8975" size="1.27" layer="95" xref="yes"/>
+<pinref part="TO-UI3" gate="1" pin="11"/>
 </segment>
 </net>
@@
 </segment>
 <segment>
-<wire x1="9.525" y1="-195.8975" x2="17.145" y2="-195.8975" width="0.1524" layer="91"/>
-<label x="17.145" y="-195.8975" size="1.27" layer="95" xref="yes"/>
-<pinref part="TO-UI3" gate="1" pin="11"/>
+<wire x1="-5.715" y1="-198.4375" x2="-10.795" y2="-198.4375" width="0.1524" layer="91"/>
+<label x="-10.795" y="-198.4375" size="1.27" layer="95" rot="R180" xref="yes"/>
+<pinref part="TO-UI3" gate="1" pin="10"/>
 </segment>
 </net>
@@
 <label x="30.48" y="-139.7" size="1.27" layer="95" rot="R90" xref="yes"/>
 </segment>
+<segment>
+<pinref part="TO-UI3" gate="1" pin="1"/>
+<wire x1="9.525" y1="-208.5975" x2="14.605" y2="-208.5975" width="0.1524" layer="91"/>
+<label x="14.605" y="-208.5975" size="1.27" layer="95" xref="yes"/>
+</segment>
 </net>
 <net name="N$27" class="0">
@@
 </segment>
 <segment>
-<pinref part="TO-UI3" gate="1" pin="6"/>
-<wire x1="-5.715" y1="-203.5175" x2="-10.795" y2="-203.5175" width="0.1524" layer="91"/>
-<label x="-10.795" y="-203.5175" size="1.27" layer="95" rot="R180" xref="yes"/>
+<pinref part="TO-UI3" gate="1" pin="3"/>
+<wire x1="9.525" y1="-206.0575" x2="14.605" y2="-206.0575" width="0.1524" layer="91"/>
+<label x="14.605" y="-206.0575" size="1.27" layer="95" xref="yes"/>
 </segment>
 </net>
@@
 </segment>
 <segment>
-<pinref part="TO-UI3" gate="1" pin="3"/>
-<wire x1="9.525" y1="-206.0575" x2="14.605" y2="-206.0575" width="0.1524" layer="91"/>
-<label x="14.605" y="-206.0575" size="1.27" layer="95" xref="yes"/>
-</segment>
-</net>
-<net name="LIPO2" class="0">
-<segment>
-<pinref part="TO-UI3" gate="1" pin="1"/>
-<wire x1="9.525" y1="-208.5975" x2="14.605" y2="-208.5975" width="0.1524" layer="91"/>
-<label x="14.605" y="-208.5975" size="1.27" layer="95" xref="yes"/>
-</segment>
-</net>
-<net name="+9V" class="0">
-<segment>
-<pinref part="SUPPLY7" gate="G$1" pin="+9V"/>
-<pinref part="TO-UI3" gate="1" pin="14"/>
-<wire x1="-9.144" y1="-188.468" x2="-9.144" y2="-193.3575" width="0.1524" layer="91"/>
-<wire x1="-9.144" y1="-193.3575" x2="-5.715" y2="-193.3575" width="0.1524" layer="91"/>
+<wire x1="-5.715" y1="-206.0575" x2="-13.335" y2="-206.0575" width="0.1524" layer="91"/>
+<label x="-13.335" y="-206.0575" size="1.27" layer="95" rot="R180" xref="yes"/>
+<pinref part="TO-UI3" gate="1" pin="4"/>
 </segment>
 </net>

Commit message: #早く仕上げろー
Parts:
- removed CN10: (no value), jst-vh:B2P-VH
- removed FET-R1, FET-R2, FET-R3, FET-R4: 100, 0@Mylibrary-main1:R-US_R0805
- removed FETR1: 4.7k, resistor-dil:4R-NEXBN8V
- removed SP-LED: (no value), led:LEDCHIPLED_0805
- removed SP-R9: 330, 0@Mylibrary-main1:R-US_R0805
- removed T1, T2: (no value), zetex:NMOS2SO8
- added 100, SP-R5: 330, 0@Mylibrary-main1:R-US_R0805
- added SP-LED1, SP-LED2: (no value), led:LEDCHIPLED_0805
- added X4, X5, X6: (no value), con-ptr500:AK500/2
- USB-POLY: value 100mA -> 400mA; device bel-fuse:0ZCH0200FF2E -> polyswitch:PTC-F0805MP
Connections:
- removed net N$17: SP-LED.C, SP-R9.2
- removed net N$29: FET-R1.1, FETR1A.2, T1A.G
- removed net N$30: FET-R2.1, FETR1B.2, T1B.G
- removed net N$32: FET-R4.1, FETR1D.2, T2B.G
- removed net N$33: FET-R3.1, FETR1C.2, T2A.G
- new net N$24: 100.2, SP-LED2.C
- new net N$5: SP-LED1.C, SP-R5.2
- net +12V: now also X6-1.KL
- net +3V3: now also SP-LED2.A, X5-1.KL
- net +5V: now also SP-LED1.A, X4-1.KL
- net +5VS: no longer SP-LED.A
- net FET1: no longer FET-R1.2
- net FET2: no longer FET-R2.2
- net FET3: no longer FET-R3.2
- net FET4: no longer FET-R4.2
- net GND: now also 100.1, SP-R5.1, X4-2.KL, X5-2.KL, X6-2.KL; no longer CN10.2, FETR1A.1, FETR1B.1, FETR1C.1, FETR1D.1, SP-R9.1, T1A.S, T1B.S, T2A.S, T2B.S
- net LED1: no longer T1A.D
- net LED2: no longer T1B.D
- net LED3: no longer T2A.D
- net LED4: no longer T2B.D
- net LIPO: no longer CN10.1

Commit message: #update 大体完成　由利倫見れたら見てw
Parts:
- removed CN2, CN3, CN4, CN5: (no value), jst-vh:B2P-VH
- added LED1, LED2, LED3, LED4: (no value), jst-vh:B3P-VH
- added SJ1, SJ2, SJ3, SJ4: (no value), jumper:SJ2WW
- renumbered CN11 to LIPO, CN6 to LED5, CN7 to LED6, CN8 to LED8, CN9 to LED7, CON1 to PING
Connections:
- removed net LED1: CN2.2
- removed net LED2: CN3.2
- removed net LED3: CN5.2
- removed net LED4: CN4.2
- new net N$17: LED3.1, SJ1.2
- new net N$32: LED1.1, SJ2.2
- new net N$37: LED4.1, SJ3.2
- new net N$40: LED2.1, SJ4.2
- net +12V: now also SJ1.1, SJ2.1, SJ3.1, SJ4.1; no longer CN2.1, CN3.1, CN4.1, CN5.1
- net +5V: now also SJ1.3, SJ2.3, SJ3.3, SJ4.3
- net FET1: now also LED1.2
- net FET2: now also LED2.2
- net FET3: now also LED3.2
- net FET4: now also LED4.2
- net GND: now also LED1.3, LED2.3, LED3.3, LED4.3

Commit message: #完成くらい
Parts:
- added CAN-R: XH-2, 0@Mylibrary-main1:XH-2
Connections:
- net CAN-H: now also CAN-R.2
- net CAN-L: now also CAN-R.1
Changed lines of the file:
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@@
 <part name="SJ4" library="jumper" library_urn="urn:adsk.eagle:library:252" deviceset="SJ2W" device="W" package3d_urn="urn:adsk.eagle:package:15476/1"/>
 <part name="GND60" library="supply1" deviceset="GND" device=""/>
+<part name="CAN-R" library="0@Mylibrary-main1" deviceset="XH-2" device=""/>
 </parts>
 <sheets>
@@
 <attribute name="VALUE" x="-180.34" y="-50.8" size="1.778" layer="96"/>
 </instance>
+<instance part="CAN-R" gate="G$1" x="-25.4" y="-175.26" smashed="yes" rot="R180">
+<attribute name="NAME" x="-22.86" y="-182.88" size="1.27" layer="95" rot="R180"/>
+<attribute name="VALUE" x="-22.86" y="-180.34" size="1.27" layer="96" rot="R180"/>
+</instance>
 </instances>
 <busses>
@@
 <label x="-33.02" y="-185.42" size="1.27" layer="95" rot="R270" xref="yes"/>
 <pinref part="CAN-R2" gate="G$1" pin="2"/>
+<pinref part="CAN-R" gate="G$1" pin="1"/>
+<wire x1="-27.94" y1="-177.8" x2="-27.94" y2="-182.88" width="0.1524" layer="91"/>
+<wire x1="-27.94" y1="-182.88" x2="-33.02" y2="-182.88" width="0.1524" layer="91"/>
+<junction x="-33.02" y="-182.88"/>
 </segment>
 <segment>
@@
 <label x="-33.02" y="-170.18" size="1.27" layer="95" rot="R90" xref="yes"/>
 <pinref part="CAN-R1" gate="G$1" pin="2"/>
+<pinref part="CAN-R" gate="G$1" pin="2"/>
+<wire x1="-27.94" y1="-172.72" x2="-33.02" y2="-172.72" width="0.1524" layer="91"/>
+<junction x="-33.02" y="-172.72"/>
 </segment>
 <segment>

Commit message: #update ほぼ完成、F7,UI,KeyHolder基板ガーバ出力済み、main基板はあとはベタ確認とシルク最終チェック。明日の夜発注する！
Parts:
- removed SP-SW2: 219-02, switch-dil:219-02
- added SJ5, SJ6: (no value), jumper:SJ
- NT-R6, NT-R7, NT-R8, NT-R9: device resistor:R-US_0207/2V -> resistor:R-US_R0805
- renumbered U$1 to 50MHZ
Connections:
- net EMERGENCY: now also TO-F7.3; no longer TO-F7.2
- net GND: now also SJ5.1, SJ6.1, TO-F7.2; no longer SP-SW2.3, SP-SW2.4, TO-F7.1
- net N$15: now also SJ6.2; no longer SP-SW2.1
- net N$26: now also SJ5.2; no longer SP-SW2.2
